Commit message: First working gazebo demo, has 2 issuses: some goals fails to be reached and the robot arm jitters while in place

File: panda_description/urdf/panda.ros2_control.xacro (robot description, xacro)
@@ -49,4 +49,20 @@
                 <state_interface name="velocity"/>
             </joint>
+                        <joint name="panda_joint7">
+                <param name="initial_position">${initial_positions['panda_joint7']}</param>
+                <command_interface name="position" />
+                <state_interface name="position"/>
+                <state_interface name="velocity"/>
+            </joint>
+            <joint name="panda_finger_joint1">
+                <command_interface name="position" />
+                <state_interface name="position"/>
+                <state_interface name="velocity"/>
+            </joint>
+            <joint name="panda_finger_joint2">
+                <command_interface name="position" />
+                <state_interface name="position"/>
+                <state_interface name="velocity"/>
+            </joint>
         </ros2_control>
     </xacro:macro>

File: panda_description/urdf/panda.urdf (robot description, URDF)
Before this commit: robot panda, 13 links, 12 joints
Links:
- link panda_leftfinger: mass 0.68 -> 0.01
- link panda_link8: mass 0.45 -> None
- link panda_rightfinger: mass 0.68 -> 0.01

Commit message: solved jitter problem, remaining collision error

File: panda_description/urdf/panda.ros2_control.xacro (robot description, xacro)
@@ -49,10 +49,4 @@
                 <state_interface name="velocity"/>
             </joint>
-                        <joint name="panda_joint7">
-                <param name="initial_position">${initial_positions['panda_joint7']}</param>
-                <command_interface name="position" />
-                <state_interface name="position"/>
-                <state_interface name="velocity"/>
-            </joint>
             <joint name="panda_finger_joint1">
                 <command_interface name="position" />

File: panda_description/urdf/panda.urdf (robot description, URDF)
Before this commit: robot panda, 13 links, 12 joints
Links:
- link panda_link8: mass None -> 0.45

File: panda_description/urdf/panda.urdf.xacro (robot description, xacro)
@@ -1,4 +1,4 @@
 <?xml version="1.0"?>
-<robot xmlns:xacro="http://www.ros.org/wiki/xacro" name="panda">
+<robot xmlns:xacro="http://www.ros.org/wiki/xacro" name="panda_arm">
     <xacro:arg name="initial_positions_file" default="initial_positions.yaml" />
     <!-- Import panda urdf file -->
