Commit message: gazebo

File: panda_description/urdf/panda.urdf (robot description, URDF)
Before this commit: robot panda, 12 links, 11 joints
Links:
- added link world
- link panda_hand: geometry collision mesh filename=package://pick_place_moveit2/panda_description/meshes/colli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; visual mesh filename=package://pick_place_moveit2/panda_description/meshes/visua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
- link panda_leftfinger: geometry collision mesh filename=package://pick_place_moveit2/panda_description/meshes/colli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; visual mesh filename=package://pick_place_moveit2/panda_description/meshes/visua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
- link panda_link0: mass None -> 3.06357; geometry collision mesh filename=package://pick_place_moveit2/panda_description/meshes/colli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 scale=1 1 1; visual mesh filename=package://pick_place_moveit2/panda_description/meshes/visua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 scale=1 1 1
- link panda_link1: geometry collision mesh filename=package://pick_place_moveit2/panda_description/meshes/colli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 scale=1 1 1; visual mesh filename=package://pick_place_moveit2/panda_description/meshes/visua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 scale=1 1 1
- link panda_link2: geometry collision mesh filename=package://pick_place_moveit2/panda_description/meshes/colli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; visual mesh filename=package://pick_place_moveit2/panda_description/meshes/visua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
- link panda_link3: geometry collision mesh filename=package://pick_place_moveit2/panda_description/meshes/colli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; visual mesh filename=package://pick_place_moveit2/panda_description/meshes/visua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
- link panda_link4: geometry collision mesh filename=package://pick_place_moveit2/panda_description/meshes/colli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; visual mesh filename=package://pick_place_moveit2/panda_description/meshes/visua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
- link panda_link5: geometry collision mesh filename=package://pick_place_moveit2/panda_description/meshes/colli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; visual mesh filename=package://pick_place_moveit2/panda_description/meshes/visua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
- link panda_link6: geometry collision mesh filename=package://pick_place_moveit2/panda_description/meshes/colli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; visual mesh filename=package://pick_place_moveit2/panda_description/meshes/visua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
- link panda_link7: geometry collision mesh filename=package://pick_place_moveit2/panda_description/meshes/colli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; visual mesh filename=package://pick_place_moveit2/panda_description/meshes/visua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
- link panda_rightfinger: geometry collision mesh filename=package://pick_place_moveit2/panda_description/meshes/colli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; visual mesh filename=package://pick_place_moveit2/panda_description/meshes/visua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
Joints:
- added joint panda_joint0: type fixed, parent world, child panda_link0, origin xyz=0 0 0 rpy=0 0 0

Commit message: gazebo

File: panda_description/urdf/panda.urdf (robot description, URDF)
Before this commit: robot panda, 13 links, 12 joints
Links:
- removed link panda_hand
- removed link panda_leftfinger
- removed link panda_link1
- removed link panda_link2
- removed link panda_link3
- removed link panda_link4
- removed link panda_link5
- removed link panda_link6
- removed link panda_link7
- removed link panda_link8
- removed link panda_rightfinger
- link panda_link0: mass 3.06357 -> 2.92; geometry collision mesh filename=/root/ws_moveit/src/pick_place_moveit2/panda_description/me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; visual mesh filename=/root/ws_moveit/src/pick_place_moveit2/panda_description/me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
Joints:
- removed joint panda_finger_joint1
- removed joint panda_finger_joint2
- removed joint panda_hand_joint
- removed joint panda_joint1
- removed joint panda_joint2
- removed joint panda_joint3
- removed joint panda_joint4
- removed joint panda_joint5
- removed joint panda_joint6
- removed joint panda_joint7
- removed joint panda_joint8

Commit message: Able to spawn link zero in gazebo

File: panda_description/urdf/panda.urdf (robot description, URDF)
Before this commit: robot panda, 2 links, 1 joints
Links:
- link panda_link0: geometry collision mesh filename=package://pick_place_moveit2/panda_description/meshes/colli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; visual mesh filename=package://pick_place_moveit2/panda_description/meshes/visua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

Commit message: Panda robot arm completely spawned in Gazebo

File: panda_description/urdf/panda.urdf (robot description, URDF)
Before this commit: robot panda, 2 links, 1 joints
Links:
- added link panda_hand, mass 0.68; collision mesh filename=package://pick_place_moveit2/panda_description/meshes/colli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; visual mesh filename=package://pick_place_moveit2/panda_description/meshes/visua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
- added link panda_leftfinger, mass 0.68; collision mesh filename=package://pick_place_moveit2/panda_description/meshes/colli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; visual mesh filename=package://pick_place_moveit2/panda_description/meshes/visua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
- added link panda_link1, mass 2.34; collision mesh filename=package://pick_place_moveit2/panda_description/meshes/colli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; visual mesh filename=package://pick_place_moveit2/panda_description/meshes/visua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
- added link panda_link2, mass 2.36; collision mesh filename=package://pick_place_moveit2/panda_description/meshes/colli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; visual mesh filename=package://pick_place_moveit2/panda_description/meshes/visua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
- added link panda_link3, mass 2.38; collision mesh filename=package://pick_place_moveit2/panda_description/meshes/colli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; visual mesh filename=package://pick_place_moveit2/panda_description/meshes/visua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
- added link panda_link4, mass 2.43; collision mesh filename=package://pick_place_moveit2/panda_description/meshes/colli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; visual mesh filename=package://pick_place_moveit2/panda_description/meshes/visua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
- added link panda_link5, mass 3.5; collision mesh filename=package://pick_place_moveit2/panda_description/meshes/colli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; visual mesh filename=package://pick_place_moveit2/panda_description/meshes/visua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
- added link panda_link6, mass 1.47; collision mesh filename=package://pick_place_moveit2/panda_description/meshes/colli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; visual mesh filename=package://pick_place_moveit2/panda_description/meshes/visua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
- added link panda_link7, mass 0.45; collision mesh filename=package://pick_place_moveit2/panda_description/meshes/colli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; visual mesh filename=package://pick_place_moveit2/panda_description/meshes/visua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
- added link panda_link8, mass 0.45
- added link panda_rightfinger, mass 0.68; collision mesh filename=package://pick_place_moveit2/panda_description/meshes/colli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; visual mesh filename=package://pick_place_moveit2/panda_description/meshes/visua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
- link panda_link0: mass 2.92 -> 3.06
Joints:
- added joint panda_finger_joint1: type prismatic, parent panda_hand, child panda_leftfinger, origin xyz=0 0 0.0584 rpy=0 0 0, axis 0 1 0, limit lower=0.0 upper=0.04 effort=20 velocity=0.2
- added joint panda_finger_joint2: type prismatic, parent panda_hand, child panda_rightfinger, origin xyz=0 0 0.0584 rpy=0 0 0, axis 0 -1 0, limit lower=0.0 upper=0.04 effort=20 velocity=0.2, mimic joint=panda_finger_joint1
- added joint panda_hand_joint: type fixed, parent panda_link8, child panda_hand, origin xyz=0 0 0 rpy=0 0 -0.785398163397
- added joint panda_joint1: type revolute, parent panda_link0, child panda_link1, origin xyz=0 0 0.333 rpy=0 0 0, axis 0 0 1, limit lower=-2.9671 upper=2.9671 effort=87 velocity=2.3925
- added joint panda_joint2: type revolute, parent panda_link1, child panda_link2, origin xyz=0 0 0 rpy=-1.57079632679 0 0, axis 0 0 1, limit lower=-1.8326 upper=1.8326 effort=87 velocity=2.3925
- added joint panda_joint3: type revolute, parent panda_link2, child panda_link3, origin xyz=0 -0.316 0 rpy=1.57079632679 0 0, axis 0 0 1, limit lower=-2.9671 upper=2.9671 effort=87 velocity=2.3925
- added joint panda_joint4: type revolute, parent panda_link3, child panda_link4, origin xyz=0.0825 0 0 rpy=1.57079632679 0 0, axis 0 0 1, limit lower=-3.1416 upper=0.0873 effort=87 velocity=2.3925
- added joint panda_joint5: type revolute, parent panda_link4, child panda_link5, origin xyz=-0.0825 0.384 0 rpy=-1.57079632679 0 0, axis 0 0 1, limit lower=-2.9671 upper=2.9671 effort=12 velocity=2.8710
- added joint panda_joint6: type revolute, parent panda_link5, child panda_link6, origin xyz=0 0 0 rpy=1.57079632679 0 0, axis 0 0 1, limit lower=-0.0873 upper=3.8223 effort=12 velocity=2.8710
- added joint panda_joint7: type revolute, parent panda_link6, child panda_link7, origin xyz=0.088 0 0 rpy=1.57079632679 0 0, axis 0 0 1, limit lower=-2.9671 upper=2.9671 effort=12 velocity=2.8710
- added joint panda_joint8: type fixed, parent panda_link7, child panda_link8, origin xyz=0 0 0.107 rpy=0 0 0, axis 0 0 0
- joint panda_joint0: axis (none) -> 0 0 0

Commit message: added laser scan to urdf file

File: panda_description/urdf/panda.urdf (robot description, URDF)
Before this commit: robot panda, 13 links, 12 joints
Links:
- added link hokuyo_link, mass 1e-5; collision box size=0.1 0.1 0.1; visual mesh filename=package://pick_place_moveit2/panda_description/meshes/hokuy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
Joints:
- added joint hokuyo_joint: type fixed, parent world, child hokuyo_link, origin xyz=0.5 0 0 rpy=0 0 0, axis 0 1 0

Commit message: added working laser scanner in gazebo

File: panda_description/urdf/panda.urdf (robot description, URDF)
Before this commit: robot panda, 14 links, 13 joints
Links:
- added link mybox, mass 0.1; collision box size=1 1 1; visual box size=1 1 1
- link hokuyo_link: mass 1e-5 -> 0.1
Joints:
- added joint mybox_joint: type fixed, parent world, child mybox, origin xyz=2 0 0 rpy=0 0 0, axis 0 1 0
- joint hokuyo_joint: origin xyz=0.5 0 0 rpy=0 0 0 -> xyz=0.2 0 0 rpy=0 0 0

Commit message: forcing all system componants to run in sim_time

File: panda_description/urdf/panda.urdf (robot description, URDF)
Before this commit: robot panda, 15 links, 14 joints
Links:
- removed link mybox
Joints:
- removed joint mybox_joint
